File: eagle/seadoo/seadoo_zs01_pcb.brd (EAGLE design)
At the start: 60 x 70 mm, 18 parts, among them Q1 IRFB7430PBF

Commit message: As sent off for first fabrication
Parts:
- added U$1, U$2: (no value), holes:3,6
- D2: device diode:D-12.5 -> 1.5KE27A:DIOAD2920W106L900D505
- moved D2 22.9 mm to (27.0, 52.0), turned to 0 degrees
- moved NTG 12.5 mm to (11.7, 41.0)
- moved C3 11.5 mm to (17.6, 49.4), turned to 0 degrees
- moved R2 10.8 mm to (31.7, 61.2), turned to 90 degrees
- moved NT+ 10.8 mm to (5.59, 41.3)
- moved C2 10.7 mm to (7.16, 49.7), turned to 180 degrees
- moved R1 3.69 mm to (25.7, 60.8), turned to 90 degrees
- moved C1 3.16 mm to (24.1, 14.5)
- moved D3 2.83 mm to (14.7, 56.6)
- moved FUSE 1.00 mm to (7.62, 21.9)
Connections:
- net N$3: now also D2.2; no longer D2.A
- net N$7: now also D2.1; no longer D2.C
Routing:
- net N$3: track 44.9 -> 76.2 mm
- net GND: track 41.5 -> 60.0 mm
- net N$6: track 41.8 -> 53.9 mm
- net N$5: track 24.0 -> 32.5 mm
- net N$7: track 51.8 -> 44.4 mm
- net BAT+_TO_MOT+: track 66.9 -> 70.6 mm
- net MOT-_TO_DRAIN: track 46.9 -> 47.9 mm
- net N$1: track 14.6 -> 13.6 mm
